File: pcb/caraccel/caraccel.kicad_sch (KiCad schematic)
At the start: 7 parts, among them J1 LESP, J2 RESP

Commit message: Fixed space in PCB 10x10 for ESP-C6. 1 inch instead of 0.9
Other:
- added sheet board_adaptor (boardadaptor.kicad_sch)
Changed lines of the file:
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@@
+		)
+	)
+	(sheet
+		(at 557.53 7.62)
+		(size 495.3 264.16)
+		(exclude_from_sim no)
+		(in_bom yes)
+		(on_board yes)
+		(dnp no)
+		(fields_autoplaced yes)
+		(stroke
+			(width 0.1524)
+			(type solid)
+		)
+		(fill
+			(color 0 0 0 0.0000)
+		)
+		(property "Sheetname" "board_adaptor"
+			(at 557.53 6.9084 0)
+			(effects
+				(font
+					(size 1.27 1.27)
+				)
+				(justify left bottom)
+			)
+		)
+		(property "Sheetfile" "boardadaptor.kicad_sch"
+			(at 557.53 272.3646 0)
+			(effects
+				(font
+					(size 1.27 1.27)
+				)
+				(justify left top)
+			)
+		)
+		(instances
+			(project "caraccel"
+				(path "/c6ba670e-d697-4bfc-9e15-b5c743a4bf76"
+					(page "2")
+				)
+			)
 		)
 	)
