File: pcb/caraccel2/caraccel2.kicad_sch (KiCad schematic)
At the start: 11 parts, among them J1 LESP, J2 RESP

Commit message: Changes in PCB
Parts:
- H1, H2, H3, H4: footprint (none) -> MountingHole:MountingHole_4.3mm_M4
Other:
- removed sheet board_adaptor
- moved on the sheet: AUXL1, AUXR1, H1, J1, J2, M8, MPU1, TFT1
